File: pcb/loraudio.kicad_pcb (KiCad board)
At the start: 2 copper layers, 70 x 50 mm, 11 parts

Commit message: Add GND net only, add design rules and mask layers
Ground net connects BAT-, PA-, PTT, AMP GND, and MIC GND.
All other connections left unassigned for now.

Co-Authored-By: Claude Opus 4.6 <noreply@anthropic.com>
Connections:
- AMP pad BCLK: I2S_BCLK -> (no net)
- AMP pad DIN: I2S_DIN -> (no net)
- AMP pad LRC: I2S_LRC -> (no net)
- AMP pad Vin: VBAT -> (no net)
- BAT pad +: VBAT -> (no net)
- MIC pad OUT: MIC_OUT -> (no net)
- MIC pad VDD: VBAT -> (no net)
- PA pad +: VBAT -> (no net)
- PTT pad 1: PTT -> (no net)
- PWR pad 1: VBAT -> (no net)
- PWR pad 2: PWR_SW -> (no net)
- SPK pad +: SPK+ -> (no net)
- SPK pad -: GND -> (no net)
Other:
- net class Default added: clearance 0.2, trace_width 0.25, via_dia 0.6, via_drill 0.3
Changed lines of the file:
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@@
     (36 "B.SilkS" user "B.Silkscreen")
     (37 "F.SilkS" user "F.Silkscreen")
+    (38 "B.Mask" user "B.Mask")
+    (39 "F.Mask" user "F.Mask")
     (44 "Edge.Cuts" user)
   )
   (setup
     (pad_to_mask_clearance 0)
+    (pcbplotparams
+      (layerselection 0x00010fc_ffffffff)
+    )
   )
   (net 0 "")
-  (net 1 "SPK+")
-  (net 2 "GND")
-  (net 3 "VBAT")
-  (net 4 "PTT")
-  (net 5 "PWR_SW")
-  (net 6 "MIC_OUT")
-  (net 7 "I2S_DIN")
-  (net 8 "I2S_BCLK")
-  (net 9 "I2S_LRC")
+  (net 1 "GND")
+  (net_class "Default" ""
+    (clearance 0.2)
+    (trace_width 0.25)
+    (via_dia 0.6)
+    (via_drill 0.3)
+  )
   (gr_rect (start 113 113) (end 183 163) (stroke (width 0.1) (type solid)) (fill none) (layer "Edge.Cuts"))
   (footprint "MountingHole_3.2mm"
@@
       (drill 0.8)
       (layers *.Cu *.Mask)
-      (net 1 "SPK+")
     )
     (pad "-" thru_hole circle
@@
       (drill 0.8)
       (layers *.Cu *.Mask)
-      (net 2 "GND")
     )
   )
@@
       (drill 0.8)
       (layers *.Cu *.Mask)
-      (net 3 "VBAT")
     )
     (pad "-" thru_hole circle
@@
       (drill 0.8)
       (layers *.Cu *.Mask)
-      (net 2 "GND")
+      (net 1 "GND")
     )
   )
@@
       (drill 0.65)
       (layers *.Cu *.Mask)
-      (net 3 "VBAT")
     )
     (pad "-" thru_hole circle
@@
       (drill 0.65)
       (layers *.Cu *.Mask)
-      (net 2 "GND")
+      (net 1 "GND")
     )
   )
@@
       (drill 0.8)
       (layers *.Cu *.Mask)
-      (net 4 "PTT")
     )
     (pad "2" thru_hole circle
@@
       (drill 0.8)
       (layers *.Cu *.Mask)
-      (net 2 "GND")
+      (net 1 "GND")
     )
   )
@@
       (drill 0.8)
       (layers *.Cu *.Mask)
-      (net 3 "VBAT")
     )
     (pad "2" thru_hole circle
@@
       (drill 0.8)
       (layers *.Cu *.Mask)
-      (net 5 "PWR_SW")
     )
   )
@@
       (drill 1.0)
       (layers *.Cu *.Mask)
-      (net 6 "MIC_OUT")
     )
     (pad "GND" thru_hole circle
@@
       (drill 1.0)
       (layers *.Cu *.Mask)
-      (net 2 "GND")
+      (net 1 "GND")
     )
     (pad "VDD" thru_hole circle
@@
       (drill 1.0)
       (layers *.Cu *.Mask)
-      (net 3 "VBAT")
     )
     (pad "AR" thru_hole circle
@@
       (drill 1.0)
       (layers *.Cu *.Mask)
-      (net 3 "VBAT")
     )
     (pad "GND" thru_hole circle
@@
       (drill 1.0)
       (layers *.Cu *.Mask)
-      (net 2 "GND")
+      (net 1 "GND")
     )
     (pad "SD" thru_hole circle
@@
       (drill 1.0)
       (layers *.Cu *.Mask)
-      (net 7 "I2S_DIN")
     )
     (pad "BCLK" thru_hole circle
@@
       (drill 1.0)
       (layers *.Cu *.Mask)
-      (net 8 "I2S_BCLK")
     )
     (pad "LRC" thru_hole circle
@@
       (drill 1.0)
       (layers *.Cu *.Mask)
-      (net 9 "I2S_LRC")
-    )
-  )
+    )
+  )
