File: pcb/loraudio.kicad_pcb (KiCad board)
At the start: 2 copper layers, 70 x 50 mm, 11 parts

Commit message: sw
Parts:
- removed PWR: , JST_PH_B2B
- added SW: , JST_PH_B2B, F.Cu at (159.0, 118.0)
Changed lines of the file:
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@@
     (layer "F.Cu")
     (at 159 118)
-    (fp_text reference "PWR" (at 0 -2.5) (layer "F.SilkS")
+    (fp_text reference "SW" (at 0 -2.5) (layer "F.SilkS")
       (effects (font (size 1 1) (thickness 0.15)))
     )
