File: pcb/loraudio.kicad_pcb (KiCad board)
At the start: 2 copper layers, 70 x 50 mm, 11 parts

Commit message: Add Heltec V4 J3 header (18-pin) to carrier board
Co-Authored-By: Claude Opus 4.6 <noreply@anthropic.com>
Parts:
- added J3: , PinHeader_1x18_P2.54mm, F.Cu at (137.6, 138.0)
Changed lines of the file:
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@@
+    )
+  )
+  (footprint "PinHeader_1x18_P2.54mm"
+    (layer "F.Cu")
+    (at 137.59 138.0)
+    (fp_text reference "J3" (at 0 -2.5) (layer "F.SilkS")
+      (effects (font (size 1 1) (thickness 0.15)))
+    )
+    (pad "GND" thru_hole circle
+      (at -21.59 0)
+      (size 1.7 1.7)
+      (drill 1.0)
+      (layers *.Cu *.Mask)
+      (net 1 "GND")
+    )
+    (pad "3V3b" thru_hole circle
+      (at -19.05 0)
+      (size 1.7 1.7)
+      (drill 1.0)
+      (layers *.Cu *.Mask)
+    )
+    (pad "3V3a" thru_hole circle
+      (at -16.509999999999998 0)
+      (size 1.7 1.7)
+      (drill 1.0)
+      (layers *.Cu *.Mask)
+    )
+    (pad "GPIO37" thru_hole circle
+      (at -13.969999999999999 0)
+      (size 1.7 1.7)
+      (drill 1.0)
+      (layers *.Cu *.Mask)
+    )
+    (pad "GPIO46" thru_hole circle
+      (at -11.43 0)
+      (size 1.7 1.7)
+      (drill 1.0)
+      (layers *.Cu *.Mask)
+    )
+    (pad "GPIO45" thru_hole circle
+      (at -8.89 0)
+      (size 1.7 1.7)
+      (drill 1.0)
+      (layers *.Cu *.Mask)
+    )
+    (pad "GPIO42" thru_hole circle
+      (at -6.35 0)
+      (size 1.7 1.7)
+      (drill 1.0)
+      (layers *.Cu *.Mask)
+    )
+    (pad "GPIO41" thru_hole circle
+      (at -3.8099999999999987 0)
+      (size 1.7 1.7)
+      (drill 1.0)
+      (layers *.Cu *.Mask)
+    )
+    (pad "GPIO40" thru_hole circle
+      (at -1.2699999999999996 0)
+      (size 1.7 1.7)
+      (drill 1.0)
+      (layers *.Cu *.Mask)
+    )
+    (pad "GPIO39" thru_hole circle
+      (at 1.2699999999999996 0)
+      (size 1.7 1.7)
+      (drill 1.0)
+      (layers *.Cu *.Mask)
+    )
+    (pad "GPIO38" thru_hole circle
+      (at 3.8099999999999987 0)
+      (size 1.7 1.7)
+      (drill 1.0)
+      (layers *.Cu *.Mask)
+    )
+    (pad "GPIO1" thru_hole circle
+      (at 6.350000000000001 0)
+      (size 1.7 1.7)
+      (drill 1.0)
+      (layers *.Cu *.Mask)
+    )
+    (pad "GPIO2" thru_hole circle
+      (at 8.89 0)
+      (size 1.7 1.7)
+      (drill 1.0)
+      (layers *.Cu *.Mask)
+    )
+    (pad "GPIO3" thru_hole circle
+      (at 11.430000000000003 0)
+      (size 1.7 1.7)
+      (drill 1.0)
+      (layers *.Cu *.Mask)
+    )
+    (pad "GPIO4" thru_hole circle
+      (at 13.970000000000002 0)
+      (size 1.7 1.7)
+      (drill 1.0)
+      (layers *.Cu *.Mask)
+    )
+    (pad "GPIO5" thru_hole circle
+      (at 16.51 0)
+      (size 1.7 1.7)
+      (drill 1.0)
+      (layers *.Cu *.Mask)
+    )
+    (pad "GPIO6" thru_hole circle
+      (at 19.05 0)
+      (size 1.7 1.7)
+      (drill 1.0)
+      (layers *.Cu *.Mask)
+    )
+    (pad "GPIO7" thru_hole circle
+      (at 21.59 0)
+      (size 1.7 1.7)
+      (drill 1.0)
+      (layers *.Cu *.Mask)
     )
   )

Commit message: Add Heltec V4 J2 header and center both rows on board
Co-Authored-By: Claude Opus 4.6 <noreply@anthropic.com>
Parts:
- added J2: , PinHeader_1x18_P2.54mm, F.Cu at (137.6, 149.4)
- moved J3 11.4 mm to (137.6, 126.6)
Changed lines of the file:
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@@
   (footprint "PinHeader_1x18_P2.54mm"
     (layer "F.Cu")
-    (at 137.59 138.0)
+    (at 137.59 126.57)
     (fp_text reference "J3" (at 0 -2.5) (layer "F.SilkS")
       (effects (font (size 1 1) (thickness 0.15)))
@@
       (at 21.59 0)
       (size 1.7 1.7)
+      (drill 1.0)
+      (layers *.Cu *.Mask)
+    )
+  )
+  (footprint "PinHeader_1x18_P2.54mm"
+    (layer "F.Cu")
+    (at 137.59 149.43)
+    (fp_text reference "J2" (at 0 -2.5) (layer "F.SilkS")
+      (effects (font (size 1 1) (thickness 0.15)))
+    )
+    (pad "GND" thru_hole circle
+      (at -21.59 0)
+      (size 1.7 1.7)
+      (drill 1.0)
+      (layers *.Cu *.Mask)
+      (net 1 "GND")
+    )
+    (pad "5V" thru_hole circle
+      (at -19.05 0)
+      (size 1.7 1.7)
+      (drill 1.0)
+      (layers *.Cu *.Mask)
+    )
+    (pad "Ve_a" thru_hole circle
+      (at -16.509999999999998 0)
+      (size 1.7 1.7)
+      (drill 1.0)
+      (layers *.Cu *.Mask)
+    )
+    (pad "Ve_b" thru_hole circle
+      (at -13.969999999999999 0)
+      (size 1.7 1.7)
+      (drill 1.0)
+      (layers *.Cu *.Mask)
+    )
+    (pad "GPIO44" thru_hole circle
+      (at -11.43 0)
+      (size 1.7 1.7)
+      (drill 1.0)
+      (layers *.Cu *.Mask)
+    )
+    (pad "GPIO43" thru_hole circle
+      (at -8.89 0)
+      (size 1.7 1.7)
+      (drill 1.0)
+      (layers *.Cu *.Mask)
+    )
+    (pad "RST" thru_hole circle
+      (at -6.35 0)
+      (size 1.7 1.7)
+      (drill 1.0)
+      (layers *.Cu *.Mask)
+    )
+    (pad "GPIO0" thru_hole circle
+      (at -3.8099999999999987 0)
+      (size 1.7 1.7)
+      (drill 1.0)
+      (layers *.Cu *.Mask)
+    )
+    (pad "GPIO36" thru_hole circle
+      (at -1.2699999999999996 0)
+      (size 1.7 1.7)
+      (drill 1.0)
+      (layers *.Cu *.Mask)
+    )
+    (pad "GPIO35" thru_hole circle
+      (at 1.2699999999999996 0)
+      (size 1.7 1.7)
+      (drill 1.0)
+      (layers *.Cu *.Mask)
+    )
+    (pad "GPIO34" thru_hole circle
+      (at 3.8099999999999987 0)
+      (size 1.7 1.7)
+      (drill 1.0)
+      (layers *.Cu *.Mask)
+    )
+    (pad "GPIO33" thru_hole circle
+      (at 6.350000000000001 0)
+      (size 1.7 1.7)
+      (drill 1.0)
+      (layers *.Cu *.Mask)
+    )
+    (pad "GPIO47" thru_hole circle
+      (at 8.89 0)
+      (size 1.7 1.7)
+      (drill 1.0)
+      (layers *.Cu *.Mask)
+    )
+    (pad "GPIO48" thru_hole circle
+      (at 11.430000000000003 0)
+      (size 1.7 1.7)
+      (drill 1.0)
+      (layers *.Cu *.Mask)
+    )
+    (pad "GPIO26" thru_hole circle
+      (at 13.970000000000002 0)
+      (size 1.7 1.7)
+      (drill 1.0)
+      (layers *.Cu *.Mask)
+    )
+    (pad "GPIO21" thru_hole circle
+      (at 16.51 0)
+      (size 1.7 1.7)
+      (drill 1.0)
+      (layers *.Cu *.Mask)
+    )
+    (pad "GPIO20" thru_hole circle
+      (at 19.05 0)
+      (size 1.7 1.7)
+      (drill 1.0)
+      (layers *.Cu *.Mask)
+    )
+    (pad "GPIO19" thru_hole circle
+      (at 21.59 0)
+      (size 1.7 1.7)
