File: pcb/loraudio.kicad_pcb (KiCad board)
At the start: 2 copper layers, 70 x 50 mm, 13 parts

Commit message: spk
Parts:
- added AMP_SPK: , PinHeader_1x2_P2.54mm, F.Cu at (172.4, 143.3)
- moved AMP 44.5 mm to (172.4, 155.0), turned to 180 degrees
- moved SPK 32.0 mm to (159.0, 118.0)
- moved BAT 8.00 mm to (127.0, 118.0)
- moved PA 8.00 mm to (135.0, 118.0)
- moved PTT 8.00 mm to (143.0, 118.0)
- moved SW 8.00 mm to (151.0, 118.0)
Connections:
- SPK pad +: (no net) -> SPK+
- SPK pad -: (no net) -> SPK-
Changed lines of the file:
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@@
   (net 3 "VSW")
   (net 4 "PTT")
-  (net 5 "3V3")
-  (net 6 "BCLK")
-  (net 7 "LRC")
-  (net 8 "DIN")
-  (net 9 "MIC_OUT")
+  (net 5 "SPK+")
+  (net 6 "SPK-")
+  (net 7 "3V3")
+  (net 8 "BCLK")
+  (net 9 "LRC")
+  (net 10 "DIN")
+  (net 11 "MIC_OUT")
   (net_class "Default" ""
     (clearance 0.2)
@@
     (layer "F.Cu")
     (at 127 118)
-    (fp_text reference "SPK" (at 0 -2.5) (layer "F.SilkS")
+    (fp_text reference "BAT" (at 0 -2.5) (layer "F.SilkS")
       (effects (font (size 1 1) (thickness 0.15)))
     )
@@
       (drill 0.8)
       (layers *.Cu *.Mask)
+      (net 1 "VBAT")
     )
     (pad "-" thru_hole circle
@@
       (drill 0.8)
       (layers *.Cu *.Mask)
-    )
-  )
-  (footprint "JST_PH_B2B"
+      (net 2 "GND")
+    )
+  )
+  (footprint "JST_SH_B2B"
     (layer "F.Cu")
     (at 135 118)
-    (fp_text reference "BAT" (at 0 -2.5) (layer "F.SilkS")
-      (effects (font (size 1 1) (thickness 0.15)))
-    )
-    (pad "+" thru_hole circle
-      (at -1.0 0)
-      (size 1.5 1.5)
-      (drill 0.8)
-      (layers *.Cu *.Mask)
-      (net 1 "VBAT")
-    )
-    (pad "-" thru_hole circle
-      (at 1.0 0)
-      (size 1.5 1.5)
-      (drill 0.8)
-      (layers *.Cu *.Mask)
-      (net 2 "GND")
-    )
-  )
-  (footprint "JST_SH_B2B"
-    (layer "F.Cu")
-    (at 143 118)
     (fp_text reference "PA" (at 0 -2.5) (layer "F.SilkS")
       (effects (font (size 1 1) (thickness 0.15)))
@@
   (footprint "JST_PH_B2B"
     (layer "F.Cu")
-    (at 151 118)
+    (at 143 118)
     (fp_text reference "PTT" (at 0 -2.5) (layer "F.SilkS")
       (effects (font (size 1 1) (thickness 0.15)))
@@
   (footprint "JST_PH_B2B"
     (layer "F.Cu")
-    (at 159 118)
+    (at 151 118)
     (fp_text reference "SW" (at 0 -2.5) (layer "F.SilkS")
       (effects (font (size 1 1) (thickness 0.15)))
@@
     )
   )
+  (footprint "JST_PH_B2B"
+    (layer "F.Cu")
+    (at 159 118)
+    (fp_text reference "SPK" (at 0 -2.5) (layer "F.SilkS")
+      (effects (font (size 1 1) (thickness 0.15)))
+    )
+    (pad "+" thru_hole circle
+      (at -1.0 0)
+      (size 1.5 1.5)
+      (drill 0.8)
+      (layers *.Cu *.Mask)
+      (net 5 "SPK+")
+    )
+    (pad "-" thru_hole circle
+      (at 1.0 0)
+      (size 1.5 1.5)
+      (drill 0.8)
+      (layers *.Cu *.Mask)
+      (net 6 "SPK-")
+    )
+  )
   (footprint "PinHeader_1x18_P2.54mm"
     (layer "F.Cu")
@@
       (drill 1.0)
       (layers *.Cu *.Mask)
-      (net 5 "3V3")
+      (net 7 "3V3")
     )
     (pad "GPIO37" thru_hole circle
@@
       (drill 1.0)
       (layers *.Cu *.Mask)
-      (net 6 "BCLK")
+      (net 8 "BCLK")
     )
     (pad "GPIO4" thru_hole circle
@@
       (drill 1.0)
       (layers *.Cu *.Mask)
-      (net 7 "LRC")
+      (net 9 "LRC")
     )
     (pad "GPIO5" thru_hole circle
@@
       (drill 1.0)
       (layers *.Cu *.Mask)
-      (net 8 "DIN")
+      (net 10 "DIN")
     )
     (pad "GPIO6" thru_hole circle
@@
       (drill 1.0)
       (layers *.Cu *.Mask)
-      (net 9 "MIC_OUT")
+      (net 11 "MIC_OUT")
     )
   )
@@
       (drill 1.0)
       (layers *.Cu *.Mask)
-      (net 9 "MIC_OUT")
+      (net 11 "MIC_OUT")
     )
     (pad "GND" thru_hole circle
@@
       (drill 1.0)
       (layers *.Cu *.Mask)
-      (net 5 "3V3")
+      (net 7 "3V3")
     )
     (pad "AR" thru_hole circle
@@
   (footprint "PinHeader_1x7_P2.54mm"
     (layer "F.Cu")
-    (at 128 158)
+    (at 172.38 155 180)
     (fp_text reference "AMP" (at 0 -2.5) (layer "F.SilkS")
       (effects (font (size 1 1) (thickness 0.15)))
@@
       (drill 1.0)
       (layers *.Cu *.Mask)
-      (net 5 "3V3")
+      (net 7 "3V3")
     )
     (pad "GND" thru_hole circle
@@
       (drill 1.0)
       (layers *.Cu *.Mask)
-      (net 8 "DIN")
+      (net 10 "DIN")
     )
     (pad "BCLK" thru_hole circle
@@
       (drill 1.0)
       (layers *.Cu *.Mask)
-      (net 6 "BCLK")
+      (net 8 "BCLK")
     )
     (pad "LRC" thru_hole circle
@@
       (drill 1.0)
       (layers *.Cu *.Mask)
-      (net 7 "LRC")
-    )
-  )
+      (net 9 "LRC")
+    )
+  )
+  (footprint "PinHeader_1x2_P2.54mm"
+    (layer "F.Cu")
+    (at 172.38 143.3 180)
+    (fp_text reference "AMP_SPK" (at 0 -2.5) (layer "F.SilkS")
+      (effects (font (size 1 1) (thickness 0.15)))
+    )
+    (pad "+" thru_hole circle
+      (at -1.27 0)
+      (size 1.7 1.7)
+      (drill 1.0)
+      (layers *.Cu *.Mask)
+      (net 5 "SPK+")
+    )
+    (pad "-" thru_hole circle
+      (at 1.27 0)
+      (size 1.7 1.7)
+      (drill 1.0)
+      (layers *.Cu *.Mask)
+      (net 6 "SPK-")
+    )
+  )

Commit message: BOM
Parts:
- removed the AMP_SPK at (172.4, 143.3)
- added AMP_SPK: , PinHeader_1x2_P3.5mm, F.Cu at (172.4, 142.0)
Changed lines of the file:
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@@
     )
   )
-  (footprint "PinHeader_1x2_P2.54mm"
+  (footprint "PinHeader_1x2_P3.5mm"
     (layer "F.Cu")
-    (at 172.38 143.3 180)
+    (at 172.38 142.046 180)
     (fp_text reference "AMP_SPK" (at 0 -2.5) (layer "F.SilkS")
       (effects (font (size 1 1) (thickness 0.15)))
     )
     (pad "+" thru_hole circle
-      (at -1.27 0)
+      (at -1.75 0)
       (size 1.7 1.7)
       (drill 1.0)
@@
     )
     (pad "-" thru_hole circle
-      (at 1.27 0)
+      (at 1.75 0)
       (size 1.7 1.7)
       (drill 1.0)

Commit message: ground plane
Routing:
- added copper zone on B.Cu, net GND
- added copper zone on F.Cu, net GND
Changed lines of the file:
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@@
+    )
+  )
+  (zone
+    (net 2)
+    (net_name "GND")
+    (layers "F.Cu" "B.Cu")
+    (hatch edge 0.5)
+    (connect_pads
+      (clearance 0.5)
+    )
+    (min_thickness 0.25)
+    (filled_areas_thickness no)
+    (fill yes
+      (thermal_gap 0.5)
+      (thermal_bridge_width 0.5)
+    )
+    (polygon
+      (pts
+        (xy 113 113) (xy 183 113) (xy 183 163) (xy 113 163)
+      )
     )
   )
