File: pcb/open-oswst.kicad_pcb (KiCad board)
At the start: 2 copper layers, 70 x 50 mm, 16 parts

Commit message: oriented correctly
Other:
- board text added: "open-oswst 77d9f79"
- board text removed: "open-oswst f0e99c9"

Commit message: correct side of board
Parts:
- moved J2 20.8 mm to (158.4, 149.4)
- moved J3 20.8 mm to (158.4, 126.6)
Other:
- board text added: "open-oswst c05cde3"
- board text removed: "open-oswst 77d9f79"
Changed lines of the file:
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@@
   )
   (gr_rect (start 113 113) (end 183 163) (stroke (width 0.1) (type solid)) (fill none) (layer "Edge.Cuts"))
-  (gr_text "open-oswst  77d9f79"
+  (gr_text "open-oswst  c05cde3"
     (at 148.0 161)
     (layer "F.SilkS")
@@
   (footprint "PinHeader_1x18_P2.54mm"
     (layer "F.Cu")
-    (at 137.59 126.57)
+    (at 158.41 126.57)
     (fp_text reference "J3" (at 0 -2.5) (layer "F.SilkS")
       (effects (font (size 1 1) (thickness 0.15)))
@@
   (footprint "PinHeader_1x18_P2.54mm"
     (layer "F.Cu")
-    (at 137.59 149.43)
+    (at 158.41 149.43)
     (fp_text reference "J2" (at 0 -2.5) (layer "F.SilkS")
       (effects (font (size 1 1) (thickness 0.15)))

Commit message: move spkr
Parts:
- moved SPK 60.0 mm to (118.0, 122.5)
- moved AMP 48.8 mm to (123.6, 155.0)
- moved AMP_SPK 48.8 mm to (123.6, 142.0)
Other:
- board text added: "open-oswst 1efcba2"
- board text removed: "open-oswst c05cde3"
Changed lines of the file:
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@@
   )
   (gr_rect (start 113 113) (end 183 163) (stroke (width 0.1) (type solid)) (fill none) (layer "Edge.Cuts"))
-  (gr_text "open-oswst  c05cde3"
+  (gr_text "open-oswst  1efcba2"
     (at 148.0 161)
     (layer "F.SilkS")
@@
   (footprint "JST_PH_B2B"
     (layer "F.Cu")
-    (at 178 122.5 90)
+    (at 118 122.5 90)
     (fp_text reference "SPK" (at 0 -2.5) (layer "F.SilkS")
       (effects (font (size 1 1) (thickness 0.15)))
@@
   (footprint "PinHeader_1x7_P2.54mm"
     (layer "F.Cu")
-    (at 172.38 155 180)
+    (at 123.62 155 180)
     (fp_text reference "AMP" (at 0 -2.5) (layer "F.SilkS")
       (effects (font (size 1 1) (thickness 0.15)))
@@
   (footprint "PinHeader_1x2_P3.5mm"
     (layer "F.Cu")
-    (at 172.38 142.046 180)
+    (at 123.62 142.046 180)
     (fp_text reference "AMP_SPK" (at 0 -2.5) (layer "F.SilkS")
       (effects (font (size 1 1) (thickness 0.15)))

Commit message: good rev
Parts:
- added HBAT: , JST_PH_B2B, F.Cu at (118.0, 122.5)
- moved PTT 24.0 mm to (170.0, 118.0)
- moved CHNL 18.0 mm to (149.0, 118.0)
- moved SPK 7.00 mm to (118.0, 129.5)
- moved VOL 4.00 mm to (160.0, 118.0)
Connections:
- AMP pad Vin: 3V3 -> Ve
- J2 pad GPIO33: BCLK -> DIN
- J2 pad GPIO47: LRC -> BCLK
- J2 pad GPIO48: DIN -> LRC
- J2 pad Ve_a: (no net) -> Ve
- J2 pad Ve_b: (no net) -> Ve
- J3 pad 3V3a: 3V3 -> (no net)
- J3 pad 3V3b: VSW -> (no net)
- J3 pad GPIO1: VOL_A -> VOL_SW
- J3 pad GPIO3: VOL_SW -> VOL_A
- J3 pad GPIO5: CHNL_A -> CHNL_SW
- J3 pad GPIO7: CHNL_SW -> CHNL_A
- MIC pad VDD: 3V3 -> Ve
Other:
- board text added: "open-oswst c31a1ce"
- board text removed: "open-oswst 1efcba2"
Changed lines of the file:
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@@
   (net 2 "GND")
   (net 3 "VSW")
-  (net 4 "PTT")
-  (net 5 "VOL_A")
-  (net 6 "VOL_B")
-  (net 7 "VOL_SW")
-  (net 8 "CHNL_A")
-  (net 9 "CHNL_B")
-  (net 10 "CHNL_SW")
+  (net 4 "CHNL_A")
+  (net 5 "CHNL_B")
+  (net 6 "CHNL_SW")
+  (net 7 "VOL_A")
+  (net 8 "VOL_B")
+  (net 9 "VOL_SW")
+  (net 10 "PTT")
   (net 11 "SPK-")
   (net 12 "SPK+")
   (net 13 "MIC_OUT")
-  (net 14 "3V3")
-  (net 15 "DIN")
-  (net 16 "LRC")
-  (net 17 "BCLK")
+  (net 14 "LRC")
+  (net 15 "BCLK")
+  (net 16 "DIN")
+  (net 17 "Ve")
   (net_class "Default" ""
     (clearance 0.2)
@@
   )
   (gr_rect (start 113 113) (end 183 163) (stroke (width 0.1) (type solid)) (fill none) (layer "Edge.Cuts"))
-  (gr_text "open-oswst  1efcba2"
+  (gr_text "open-oswst  c31a1ce"
     (at 148.0 161)
     (layer "F.SilkS")
@@
     )
   )
-  (footprint "JST_PH_B2B"
-    (layer "F.Cu")
-    (at 146 118)
-    (fp_text reference "PTT" (at 0 -2.5) (layer "F.SilkS")
-      (effects (font (size 1 1) (thickness 0.15)))
-    )
-    (pad "1" thru_hole circle
-      (at -1.0 0)
-      (size 1.5 1.5)
-      (drill 0.8)
-      (layers *.Cu *.Mask)
-      (net 4 "PTT")
-    )
-    (pad "2" thru_hole circle
-      (at 1.0 0)
-      (size 1.5 1.5)
-      (drill 0.8)
-      (layers *.Cu *.Mask)
-      (net 2 "GND")
-    )
-  )
   (footprint "JST_PH_B4B"
     (layer "F.Cu")
-    (at 156 118)
-    (fp_text reference "VOL" (at 0 -2.5) (layer "F.SilkS")
+    (at 149 118)
+    (fp_text reference "CHNL" (at 0 -2.5) (layer "F.SilkS")
       (effects (font (size 1 1) (thickness 0.15)))
     )
@@
       (drill 0.8)
       (layers *.Cu *.Mask)
-      (net 5 "VOL_A")
+      (net 4 "CHNL_A")
     )
     (pad "B" thru_hole circle
@@
       (drill 0.8)
       (layers *.Cu *.Mask)
-      (net 6 "VOL_B")
+      (net 5 "CHNL_B")
     )
     (pad "SW" thru_hole circle
@@
       (drill 0.8)
       (layers *.Cu *.Mask)
-      (net 7 "VOL_SW")
+      (net 6 "CHNL_SW")
     )
     (pad "GND" thru_hole circle
@@
   (footprint "JST_PH_B4B"
     (layer "F.Cu")
-    (at 167 118)
-    (fp_text reference "CHNL" (at 0 -2.5) (layer "F.SilkS")
+    (at 160 118)
+    (fp_text reference "VOL" (at 0 -2.5) (layer "F.SilkS")
       (effects (font (size 1 1) (thickness 0.15)))
     )
@@
       (drill 0.8)
       (layers *.Cu *.Mask)
-      (net 8 "CHNL_A")
+      (net 7 "VOL_A")
     )
     (pad "B" thru_hole circle
@@
       (drill 0.8)
       (layers *.Cu *.Mask)
-      (net 9 "CHNL_B")
+      (net 8 "VOL_B")
     )
     (pad "SW" thru_hole circle
@@
       (drill 0.8)
       (layers *.Cu *.Mask)
-      (net 10 "CHNL_SW")
+      (net 9 "VOL_SW")
     )
     (pad "GND" thru_hole circle
@@
   (footprint "JST_PH_B2B"
     (layer "F.Cu")
+    (at 170 118)
+    (fp_text reference "PTT" (at 0 -2.5) (layer "F.SilkS")
+      (effects (font (size 1 1) (thickness 0.15)))
+    )
+    (pad "1" thru_hole circle
+      (at -1.0 0)
+      (size 1.5 1.5)
+      (drill 0.8)
+      (layers *.Cu *.Mask)
+      (net 10 "PTT")
+    )
+    (pad "2" thru_hole circle
+      (at 1.0 0)
+      (size 1.5 1.5)
+      (drill 0.8)
+      (layers *.Cu *.Mask)
+      (net 2 "GND")
+    )
+  )
+  (footprint "JST_PH_B2B"
+    (layer "F.Cu")
     (at 118 122.5 90)
+    (fp_text reference "HBAT" (at 0 -2.5) (layer "F.SilkS")
+      (effects (font (size 1 1) (thickness 0.15)))
+    )
+    (pad "+" thru_hole circle
+      (at -1.0 0)
+      (size 1.5 1.5)
+      (drill 0.8)
+      (layers *.Cu *.Mask)
+      (net 3 "VSW")
+    )
+    (pad "-" thru_hole circle
+      (at 1.0 0)
+      (size 1.5 1.5)
+      (drill 0.8)
+      (layers *.Cu *.Mask)
+      (net 2 "GND")
+    )
+  )
+  (footprint "JST_PH_B2B"
+    (layer "F.Cu")
+    (at 118 129.5 90)
     (fp_text reference "SPK" (at 0 -2.5) (layer "F.SilkS")
       (effects (font (size 1 1) (thickness 0.15)))
@@
       (drill 1.0)
       (layers *.Cu *.Mask)
-      (net 10 "CHNL_SW")
+      (net 4 "CHNL_A")
     )
     (pad "GPIO6" thru_hole circle
@@
       (drill 1.0)
       (layers *.Cu *.Mask)
-      (net 9 "CHNL_B")
+      (net 5 "CHNL_B")
     )
     (pad "GPIO5" thru_hole circle
@@
       (drill 1.0)
       (layers *.Cu *.Mask)
-      (net 8 "CHNL_A")
+      (net 6 "CHNL_SW")
     )
     (pad "GPIO4" thru_hole circle
@@
       (drill 1.0)
       (layers *.Cu *.Mask)
-      (net 7 "VOL_SW")
+      (net 7 "VOL_A")
     )
     (pad "GPIO2" thru_hole circle
@@
       (drill 1.0)
       (layers *.Cu *.Mask)
-      (net 6 "VOL_B")
+      (net 8 "VOL_B")
     )
     (pad "GPIO1" thru_hole circle
@@
       (drill 1.0)
       (layers *.Cu *.Mask)
-      (net 5 "VOL_A")
+      (net 9 "VOL_SW")
     )
     (pad "GPIO38" thru_hole circle
@@
       (drill 1.0)
       (layers *.Cu *.Mask)
-      (net 14 "3V3")
     )
     (pad "3V3b" thru_hole circle
@@
       (drill 1.0)
       (layers *.Cu *.Mask)
-      (net 3 "VSW")
     )
     (pad "GND" thru_hole circle
@@
       (drill 1.0)
       (layers *.Cu *.Mask)
-      (net 15 "DIN")
+      (net 14 "LRC")
     )
     (pad "GPIO47" thru_hole circle
@@
       (drill 1.0)
       (layers *.Cu *.Mask)
-      (net 16 "LRC")
+      (net 15 "BCLK")
     )
     (pad "GPIO33" thru_hole circle
@@
       (drill 1.0)
       (layers *.Cu *.Mask)
-      (net 17 "BCLK")
+      (net 16 "DIN")
     )
     (pad "GPIO34" thru_hole circle
@@
       (drill 1.0)
       (layers *.Cu *.Mask)
-      (net 4 "PTT")
+      (net 10 "PTT")
     )
     (pad "RST" thru_hole circle
@@
       (drill 1.0)
       (layers *.Cu *.Mask)
+      (net 17 "Ve")
     )
     (pad "Ve_a" thru_hole circle
@@
       (drill 1.0)
       (layers *.Cu *.Mask)
+      (net 17 "Ve")
     )
     (pad "5V" thru_hole circle
@@
       (drill 1.0)
       (layers *.Cu *.Mask)
-      (net 14 "3V3")
+      (net 17 "Ve")
     )
     (pad "GAIN" thru_hole circle
@@
       (drill 1.0)
       (layers *.Cu *.Mask)
-      (net 14 "3V3")
+      (net 17 "Ve")
     )
     (pad "GND" thru_hole circle
@@
       (drill 1.0)
       (layers *.Cu *.Mask)
-      (net 15 "DIN")
+      (net 16 "DIN")
     )
     (pad "BCLK" thru_hole circle
@@
       (drill 1.0)
       (layers *.Cu *.Mask)
-      (net 17 "BCLK")
+      (net 15 "BCLK")
     )
     (pad "LRC" thru_hole circle
@@
       (drill 1.0)
       (layers *.Cu *.Mask)
-      (net 16 "LRC")
-    )
-  )
+      (net 14 "LRC")
+    )
+  )

Commit message: good rev
Other:
- net class Power added: clearance 0.2, trace_width 0.5, via_dia 0.8, via_drill 0.4
- board text added: "open-oswst b9fa6db"
- board text removed: "open-oswst c31a1ce"
Changed lines of the file:
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@@
     (via_drill 0.3)
   )
+  (net_class "Power" "Battery rail — 800mA peak during TX"
+    (clearance 0.2)
+    (trace_width 0.5)
+    (via_dia 0.8)
+    (via_drill 0.4)
+    (add_net "VBAT")
+    (add_net "VSW")
+  )
   (gr_rect (start 113 113) (end 183 163) (stroke (width 0.1) (type solid)) (fill none) (layer "Edge.Cuts"))
-  (gr_text "open-oswst  c31a1ce"
+  (gr_text "open-oswst  b9fa6db"
     (at 148.0 161)
     (layer "F.SilkS")

Commit message: rev5 :(
Other:
- board text added: "open-oswst 4d31d95"
- board text removed: "open-oswst b9fa6db"
Changed lines of the file:
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@@
   )
   (gr_rect (start 113 113) (end 183 163) (stroke (width 0.1) (type solid)) (fill none) (layer "Edge.Cuts"))
-  (gr_text "open-oswst  b9fa6db"
+  (gr_text "open-oswst  4d31d95"
     (at 148.0 161)
     (layer "F.SilkS")
@@
       (effects (font (size 1 1) (thickness 0.15)))
     )
-    (pad "GND" thru_hole circle
+    (pad "AR" thru_hole circle
       (at -5.08 0)
       (size 1.7 1.7)
       (drill 1.0)
       (layers *.Cu *.Mask)
-      (net 2 "GND")
-    )
-    (pad "VDD" thru_hole circle
+    )
+    (pad "OUT" thru_hole circle
       (at -2.54 0)
       (size 1.7 1.7)
       (drill 1.0)
       (layers *.Cu *.Mask)
-      (net 17 "Ve")
+      (net 13 "MIC_OUT")
     )
     (pad "GAIN" thru_hole circle
@@
       (layers *.Cu *.Mask)
     )
-    (pad "OUT" thru_hole circle
+    (pad "VDD" thru_hole circle
       (at 2.54 0)
       (size 1.7 1.7)
       (drill 1.0)
       (layers *.Cu *.Mask)
-      (net 13 "MIC_OUT")
-    )
-    (pad "AR" thru_hole circle
+      (net 17 "Ve")
+    )
+    (pad "GND" thru_hole circle
       (at 5.08 0)
       (size 1.7 1.7)
       (drill 1.0)
       (layers *.Cu *.Mask)
-    )
-  )
+      (net 2 "GND")
+    )
+  )
